Commit message: r200 camera minor name change

File: urdf/cameras/rgbd/realsense_r200.urdf.xacro (robot description, xacro)
@@ -3,5 +3,5 @@
      <xacro:macro name="sensor_realsense_r200" params="prefix:='' parent *origin visualize:=false">
           <!-- Camera link -->
-          <link name="${prefix}rs200_camera">
+          <link name="${prefix}r200_camera">
                <visual>
                     <origin rpy="0 0 0" xyz="0 0 0"/>
@@ -30,5 +30,5 @@
           <joint name="${prefix}realsense_joint" type="fixed">
                <parent link="${parent}"/>
-               <child link="${prefix}rs200_camera"/>
+               <child link="${prefix}r200_camera"/>
                <xacro:insert_block name="origin"/>
           </joint>
@@ -40,20 +40,20 @@
           <!-- Joints positioning the virtual links with respect to the camera main link-->
           <joint name="${prefix}color_joint" type="fixed">
-               <parent link="${prefix}rs200_camera" />
+               <parent link="${prefix}r200_camera" />
                <child link="${prefix}color" />
                <origin xyz="0 -0.046 0.004" rpy="${pi/2} ${pi} ${pi/2}"/>
           </joint>
           <joint name="${prefix}depth_joint" type="fixed">
-               <parent link="${prefix}rs200_camera" />
+               <parent link="${prefix}r200_camera" />
                <child link="${prefix}depth" />
                <origin xyz="0 -0.03 0.004" rpy="0 0 0"/>
           </joint>
           <joint name="${prefix}ired1_joint" type="fixed">
-               <parent link="${prefix}rs200_camera" />
+               <parent link="${prefix}r200_camera" />
                <child link="${prefix}ired1" />
                <origin xyz="0 -0.06 0.004" rpy="0 0 0"/>
           </joint>
           <joint name="${prefix}ired2_joint" type="fixed">
-               <parent link="${prefix}rs200_camera" />
+               <parent link="${prefix}r200_camera" />
                <child link="${prefix}ired2" />
                <origin xyz="0 0.01 0.004" rpy="0 0 0"/>
@@ -66,5 +66,5 @@
           </gazebo>
           <!-- Load parameters to model's main link-->
-          <gazebo reference="${prefix}rs200_camera">
+          <gazebo reference="${prefix}r200_camera">
                <!-- ================== Color Camera =================== -->
                <sensor name="color" type="camera">
