Commit message: fixed references in urdf files. renamed urdf files and internals. mesh directory restructured

File: urdf/all_sensors.urdf.xacro (robot description, xacro)
@@ -5,20 +5,20 @@
                          	Cameras
      ========================================================= -->
-	<xacro:include filename="$(find terrasentia_sensors)/urdf/cameras/camera_sensors.urdf.xacro" />
+	<xacro:include filename="$(find gazebo_sensor_collection)/urdf/cameras/camera_sensors.urdf.xacro" />
 	<!-- ====================================================
 						GPS
 	========================================================= -->
-	<xacro:include filename="$(find terrasentia_sensors)/urdf/gps/gps_sensors.urdf.xacro" />
+	<xacro:include filename="$(find gazebo_sensor_collection)/urdf/gps/gps_sensors.urdf.xacro" />
 	<!-- ====================================================
                          	LiDAR
      ========================================================= -->
-	<xacro:include filename="$(find terrasentia_sensors)/urdf/lidars/lidar_sensors.urdf.xacro" />
+	<xacro:include filename="$(find gazebo_sensor_collection)/urdf/lidars/lidar_sensors.urdf.xacro" />
 	<!-- ====================================================
                          	Motion
      ========================================================= -->
-	<xacro:include filename="$(find terrasentia_sensors)/urdf/motion/motion_sensors.urdf.xacro" />
+	<xacro:include filename="$(find gazebo_sensor_collection)/urdf/motion/motion_sensors.urdf.xacro" />
 	<!-- ====================================================
                          	Misc
      ========================================================= -->
-	<xacro:include filename="$(find terrasentia_sensors)/urdf/misc/misc_sensors.urdf.xacro" />
+	<xacro:include filename="$(find gazebo_sensor_collection)/urdf/misc/misc_sensors.urdf.xacro" />
 </robot>

File: urdf/cameras/camera_sensors.urdf.xacro (robot description, xacro)
@@ -5,25 +5,25 @@
      ========================================================= -->
 	<!-- Axis p5512 -->
-	<xacro:include filename="$(find terrasentia_sensors)/urdf/cameras/rgb/axis_p5512.urdf.xacro" />
+	<xacro:include filename="$(find gazebo_sensor_collection)/urdf/cameras/rgb/axis_p5512.urdf.xacro" />
 	<!-- Axis m5013 -->
-	<xacro:include filename="$(find terrasentia_sensors)/urdf/cameras/rgb/axis_m5013.urdf.xacro" />
+	<xacro:include filename="$(find gazebo_sensor_collection)/urdf/cameras/rgb/axis_m5013.urdf.xacro" />
 	<!-- uEye CP Gige -->
-	<xacro:include filename="$(find terrasentia_sensors)/urdf/cameras/rgb/ueye_cp_gige.urdf.xacro" />
+	<xacro:include filename="$(find gazebo_sensor_collection)/urdf/cameras/rgb/ueye_cp_gige.urdf.xacro" />
 	<!-- ELP USB Camera w/ Normal Lens -->
-	<xacro:include filename="$(find terrasentia_sensors)/urdf/cameras/rgb/elp_usb_camera.urdf.xacro" />
+	<xacro:include filename="$(find gazebo_sensor_collection)/urdf/cameras/rgb/elp_usb_camera.urdf.xacro" />
 	<!-- ====================================================
                          	RGBD
      ========================================================= -->
 	<!-- Asus Xtion PRO -->
-	<xacro:include filename="$(find terrasentia_sensors)/urdf/cameras/rgbd/asus_xtion_pro.urdf.xacro" />
+	<xacro:include filename="$(find gazebo_sensor_collection)/urdf/cameras/rgbd/asus_xtion_pro.urdf.xacro" />
 	<!-- Kinect -->
-	<xacro:include filename="$(find terrasentia_sensors)/urdf/cameras/rgbd/kinect.urdf.xacro" />
+	<xacro:include filename="$(find gazebo_sensor_collection)/urdf/cameras/rgbd/kinect.urdf.xacro" />
 	<!-- KinectV2 -->
-	<xacro:include filename="$(find terrasentia_sensors)/urdf/cameras/rgbd/kinectv2.urdf.xacro" />
+	<xacro:include filename="$(find gazebo_sensor_collection)/urdf/cameras/rgbd/kinectv2.urdf.xacro" />
 	<!-- Orbbec Astra -->
-	<xacro:include filename="$(find terrasentia_sensors)/urdf/cameras/rgbd/orbbec_astra.urdf.xacro" />
+	<xacro:include filename="$(find gazebo_sensor_collection)/urdf/cameras/rgbd/orbbec_astra.urdf.xacro" />
 	<!-- Fotonic E Series -->
-	<xacro:include filename="$(find terrasentia_sensors)/urdf/cameras/rgbd/fotonic_e.urdf.xacro" />
+	<xacro:include filename="$(find gazebo_sensor_collection)/urdf/cameras/rgbd/fotonic_e.urdf.xacro" />
 	<!-- Intel Realsense R200 -->
-	<xacro:include filename="$(find terrasentia_sensors)/urdf/cameras/rgbd/realsense_r200.urdf.xacro" />
+	<xacro:include filename="$(find gazebo_sensor_collection)/urdf/cameras/rgbd/realsense_r200.urdf.xacro" />
 </robot>

File: urdf/cameras/rgb/axis_m5013.urdf.xacro (robot description, xacro)
@@ -1,5 +1,5 @@
 <?xml version="1.0"?>
 <robot xmlns:xacro="http://ros.org/wiki/xacro" name="sensor_axis_m5013">
-     <xacro:include filename="$(find terrasentia_sensors)/urdf/includes/materials.urdf.xacro"/>
+     <xacro:include filename="$(find gazebo_sensor_collection)/urdf/includes/materials.urdf.xacro"/>
      <xacro:property name="ptz_joint_effort_limit" value="100.0"/>
      <xacro:property name="ptz_joint_velocity_limit" value="100.0"/>
@@ -25,5 +25,5 @@
                     <origin xyz="0 0 0" rpy="0 ${M_PI/2} 0"/>
                     <geometry>
-                         <mesh filename="package://terrasentia_sensors/meshes/axis_m5013.dae" scale="1.0 1.0 1.0"/>
+                         <mesh filename="package://gazebo_sensor_collection/meshes/cameras/axis/axis_m5013.dae" scale="1.0 1.0 1.0"/>
                     </geometry>
                     <xacro:color_material color="${color}"/>
@@ -32,5 +32,5 @@
                     <origin xyz="0.0 0.0 0" rpy="0 ${M_PI/2} 0"/>
                     <geometry>
-                         <mesh filename="package://terrasentia_sensors/meshes/axis_m5013.stl" scale="1.0 1.0 1.0"/>
+                         <mesh filename="package://gazebo_sensor_collection/meshes/cameras/axis/axis_m5013.stl" scale="1.0 1.0 1.0"/>
                     </geometry>
                </collision>

File: urdf/cameras/rgb/axis_p5512.urdf.xacro (robot description, xacro)
@@ -1,5 +1,5 @@
 <?xml version="1.0"?>
 <robot xmlns:xacro="http://ros.org/wiki/xacro" name="sensor_axis_p5512">
-     <xacro:include filename="$(find terrasentia_sensors)/urdf/includes/materials.urdf.xacro"/>
+     <xacro:include filename="$(find gazebo_sensor_collection)/urdf/includes/materials.urdf.xacro"/>
      <xacro:property name="ptz_joint_effort_limit" value="100.0"/>
      <xacro:property name="ptz_joint_velocity_limit" value="100.0"/>
@@ -25,5 +25,5 @@
                     <origin xyz="-0.3 0.0 -0.03" rpy="0 ${M_PI/2} 0"/>
                     <geometry>
-                         <mesh filename="package://terrasentia_sensors/meshes/axis_p5512.stl" scale="1.0 1.0 1.0"/>
+                         <mesh filename="package://gazebo_sensor_collection/meshes/cameras/axis/axis_p5512.stl" scale="1.0 1.0 1.0"/>
                     </geometry>
                     <xacro:color_material color="${color}"/>
@@ -33,5 +33,5 @@
                     <!-- because the origin of the mesh file is not at the "center" of the model-->
                     <geometry>
-                         <mesh filename="package://terrasentia_sensors/meshes/axis_p5512.stl" scale="1.0 1.0 1.0"/>
+                         <mesh filename="package://gazebo_sensor_collection/meshes/cameras/axis/axis_p5512.stl" scale="1.0 1.0 1.0"/>
                     </geometry>
                </collision>

File: urdf/cameras/rgb/elp_usb_camera.urdf.xacro (robot description, xacro)
@@ -1,5 +1,5 @@
 <?xml version="1.0"?>
 <robot xmlns:xacro="http://ros.org/wiki/xacro">
-     <xacro:include filename="$(find terrasentia_sensors)/urdf/includes/materials.urdf.xacro"/>
+     <xacro:include filename="$(find gazebo_sensor_collection)/urdf/includes/materials.urdf.xacro"/>
      <xacro:macro name="sensor_elp_usb_cam" params="name parent *origin color">
           <joint name="${name}_joint" type="fixed">
@@ -19,5 +19,5 @@
                          <xacro:color_material color="${color}"/>
                          <geometry>
-                              <mesh filename="package://terrasentia_sensors/meshes/board_camera.dae" scale="1.0 1.0 1.0"/>
+                              <mesh filename="package://gazebo_sensor_collection/meshes/cameras/misc/board_camera.dae" scale="1.0 1.0 1.0"/>
                          </geometry>
                </visual>
@@ -25,5 +25,5 @@
                     <origin xyz="0.0 0.0 0.0" rpy="0 0 0"/>
                     <geometry>
-                         <mesh filename="package://terrasentia_sensors/meshes/board_camera.dae" scale="1.0 1.0 1.0"/>
+                         <mesh filename="package://gazebo_sensor_collection/meshes/cameras/misc/board_camera.dae" scale="1.0 1.0 1.0"/>
                     </geometry>
                </collision>

File: urdf/cameras/rgb/ueye_cp_gige.urdf.xacro (robot description, xacro)
@@ -1,5 +1,5 @@
 <?xml version="1.0"?>
 <robot xmlns:xacro="http://ros.org/wiki/xacro">
-     <xacro:include filename="$(find terrasentia_sensors)/urdf/includes/materials.urdf.xacro"/>
+     <xacro:include filename="$(find gazebo_sensor_collection)/urdf/includes/materials.urdf.xacro"/>
      <xacro:macro name="sensor_ueye_cp_gige" params="name parent *origin color">
           <joint name="${name}_joint" type="fixed">
@@ -19,5 +19,5 @@
                          <xacro:color_material color="${color}"/>
                          <geometry>
-                              <mesh filename="package://terrasentia_sensors/meshes/ueye_cp_gige.stl" scale="1.0 1.0 1.0"/>
+                              <mesh filename="package://gazebo_sensor_collection/meshes/cameras/ids/ueye_cp_gige.stl" scale="1.0 1.0 1.0"/>
                          </geometry>
                </visual>
@@ -25,5 +25,5 @@
                     <origin xyz="0.0 0.0 0.0" rpy="0 0 0"/>
                     <geometry>
-                         <mesh filename="package://terrasentia_sensors/meshes/ueye_cp_gige.stl" scale="1.0 1.0 1.0"/>
+                         <mesh filename="package://gazebo_sensor_collection/meshes/cameras/ids/ueye_cp_gige.stl" scale="1.0 1.0 1.0"/>
                     </geometry>
                </collision>

File: urdf/cameras/rgbd/asus_xtion_pro.urdf.xacro (robot description, xacro)
@@ -1,5 +1,5 @@
 <?xml version="1.0"?>
 <robot name="sensor_asus_xtion_pro" xmlns:xacro="http://ros.org/wiki/xacro">
-     <xacro:include filename="$(find terrasentia_sensors)/urdf/includes/materials.urdf.xacro"/>
+     <xacro:include filename="$(find gazebo_sensor_collection)/urdf/includes/materials.urdf.xacro"/>
      <xacro:property name="asus_xtion_scale" value="1.0"/>
      <xacro:property name="asus_xtion_pro_depth_rel_rgb_py" value="0.0270" />
@@ -40,5 +40,5 @@
                     <origin xyz="-0.01 0 0" rpy="${-M_PI/2} -${M_PI} ${-M_PI/2}"/>
                     <geometry>
-                         <mesh filename="package://terrasentia_sensors/meshes/asus_xtion_pro_live.dae" scale="${asus_xtion_scale} ${asus_xtion_scale} ${asus_xtion_scale}"/>
+                         <mesh filename="package://gazebo_sensor_collection/meshes/cameras/asus/asus_xtion_pro_live.dae" scale="${asus_xtion_scale} ${asus_xtion_scale} ${asus_xtion_scale}"/>
                     </geometry>
                     <xacro:color_material color="${color}"/>

File: urdf/cameras/rgbd/fotonic_e.urdf.xacro (robot description, xacro)
@@ -1,5 +1,5 @@
 <?xml version="1.0"?>
 <robot name="sensor_fotonic" xmlns:xacro="http://ros.org/wiki/xacro">
-	<xacro:include filename="$(find terrasentia_sensors)/urdf/includes/materials.urdf.xacro"/>
+	<xacro:include filename="$(find gazebo_sensor_collection)/urdf/includes/materials.urdf.xacro"/>
 	<xacro:macro name="sensor_fotonic" params="name parent *origin color">
 		<joint name="${name}_joint" type="fixed">
@@ -18,5 +18,5 @@
 				<origin xyz="0.0 0.0 -0.04" rpy="0 0 0" /> <!-- to center the .dae model -->
 				<geometry>
-					<mesh filename= "package://terrasentia_sensors/meshes/fotonic_e.stl" scale="1.0 1.0 1.0"/>
+					<mesh filename= "package://gazebo_sensor_collection/meshes/cameras/acroname/fotonic_e.stl" scale="1.0 1.0 1.0"/>
 				</geometry>
 				<xacro:color_material color="${color}"/>
@@ -25,5 +25,5 @@
 				<origin xyz="0.0 0 -0.04" rpy="0 0 0" />
 				<geometry>
-					<mesh filename= "package://terrasentia_sensors/meshes/fotonic_e.stl" scale="1.0 1.0 1.0"/>
+					<mesh filename= "package://gazebo_sensor_collection/meshes/cameras/acroname/fotonic_e.stl" scale="1.0 1.0 1.0"/>
 				</geometry>
 			</collision>

File: urdf/cameras/rgbd/kinect.urdf.xacro (robot description, xacro)
@@ -1,5 +1,5 @@
 <?xml version="1.0"?>
 <robot name="sensor_kinect" xmlns:xacro="http://ros.org/wiki/xacro">
-	<xacro:include filename="$(find terrasentia_sensors)/urdf/includes/materials.urdf.xacro"/>
+	<xacro:include filename="$(find gazebo_sensor_collection)/urdf/includes/materials.urdf.xacro"/>
 	<xacro:property name="M_PI" value="3.1415926535897931" />
 	<xacro:property name="cam_px" value="-0.087" />
@@ -43,5 +43,5 @@
 				<origin xyz="0 0 0" rpy="0 0 ${M_PI/2}"/>
 				<geometry>
-					<mesh filename="package://terrasentia_sensors/meshes/kinect.dae"/>
+					<mesh filename="package://gazebo_sensor_collection/meshes/cameras/microsoft/kinect.dae"/>
 				</geometry>
 				<xacro:color_material color="${color}"/>

File: urdf/cameras/rgbd/kinectv2.urdf.xacro (robot description, xacro)
@@ -1,5 +1,5 @@
 <?xml version="1.0"?>
 <robot name="sensor_kinectv2" xmlns:xacro="http://ros.org/wiki/xacro">
-     <xacro:include filename="$(find terrasentia_sensors)/urdf/includes/materials.urdf.xacro"/>
+     <xacro:include filename="$(find gazebo_sensor_collection)/urdf/includes/materials.urdf.xacro"/>
      <xacro:property name="M_PI" value="3.1415926535897931" />
      <xacro:property name="cam_px" value="-0.087" />
@@ -49,8 +49,8 @@
                     <geometry>
                          <xacro:if value="${base}">
-                              <mesh filename="package://terrasentia_sensors/meshes/kinectv2.dae"/>
+                              <mesh filename="package://gazebo_sensor_collection/meshes/cameras/microsoft/kinectv2.dae"/>
                          </xacro:if>
                          <xacro:unless value="${base}">
-                              <mesh filename="package://terrasentia_sensors/meshes/kinectv2_nobase.dae"/>
+                              <mesh filename="package://gazebo_sensor_collection/meshes/cameras/microsoft/kinectv2_nobase.dae"/>
                          </xacro:unless>
                     </geometry>

File: urdf/cameras/rgbd/orbbec_astra.urdf.xacro (robot description, xacro)
@@ -1,5 +1,5 @@
 <?xml version="1.0"?>
 <robot name="sensor_orbbec_astra" xmlns:xacro="http://ros.org/wiki/xacro">
-     <xacro:include filename="$(find terrasentia_sensors)/urdf/includes/materials.urdf.xacro"/>
+     <xacro:include filename="$(find gazebo_sensor_collection)/urdf/includes/materials.urdf.xacro"/>
      <xacro:property name="orbbec_astra_scale" value="1.0"/>
      <!-- RGB sensor - cam -->
@@ -46,5 +46,5 @@
                     <origin xyz="0 0 0" rpy="0 0 0"/>
                     <geometry>
-                         <mesh filename="package://terrasentia_sensors/meshes/orbbec_astra.dae" scale="${orbbec_astra_scale} ${orbbec_astra_scale} ${orbbec_astra_scale}"/>
+                         <mesh filename="package://gazebo_sensor_collection/meshes/cameras/orbbec/orbbec_astra.dae" scale="${orbbec_astra_scale} ${orbbec_astra_scale} ${orbbec_astra_scale}"/>
                     </geometry>
                     <xacro:color_material color="${color}"/>

File: urdf/cameras/rgbd/realsense_r200.urdf.xacro (robot description, xacro)
@@ -7,5 +7,5 @@
                     <origin rpy="0 0 0" xyz="0 0 0"/>
                     <geometry>
-                         <mesh filename="package://terrasentia_sensors/meshes/realsense_r200/realsense.dae"/>
+                         <mesh filename="package://gazebo_sensor_collection/meshes/cameras/intel/realsense_r200.dae"/>
                     </geometry>
                </visual>

File: urdf/gps/gps_quad.urdf.xacro (robot description, xacro)
@@ -1,5 +1,5 @@
 <?xml version="1.0"?>
-<robot name="sensor_gps" xmlns:xacro="http://ros.org/wiki/xacro">
-	<xacro:include filename="$(find terrasentia_sensors)/urdf/includes/materials.urdf.xacro"/>
+<robot name="sensor_gps_quad" xmlns:xacro="http://ros.org/wiki/xacro">
+	<xacro:include filename="$(find gazebo_sensor_collection)/urdf/includes/materials.urdf.xacro"/>
   	<xacro:macro name="sensor_gps_quad" params="name parent *origin color ref_lat ref_long ref_head drift vel_drift noise vel_noise update_rate">
 		<joint name="${name}_joint" type="revolute">
@@ -20,5 +20,5 @@
 				<origin rpy="0 0 0" xyz="0 0 0"/>
 				<geometry>
-					<mesh filename="package://terrasentia_sensors/meshes/antenna_3GO16.stl" scale="1.0 1.0 1.0"/>
+					<mesh filename="package://gazebo_sensor_collection/meshes/gps/antenna_3GO16.stl" scale="1.0 1.0 1.0"/>
 				</geometry>
 				<xacro:color_material color="${color}"/>
@@ -40,5 +40,5 @@
 				<alwaysOn>1</alwaysOn>
 				<updateRate>${update_rate}</updateRate>
-				<bodyName>${name}_link</bodyName> <!-- must be the link of the gps device, not the base_link or base_footprint -->
+				<bodyName>${name}_link</bodyName>
 				<!-- <frameId>${name}_link</frameId> -->
 				<topicName>${name}</topicName>
@@ -54,4 +54,3 @@
 		</gazebo>
 	</xacro:macro>
-	<!--<xacro:include filename="$(find terrasentia_sensors)/config/dropouts.xml"/>-->
 </robot>

File: urdf/gps/gps_sensors.urdf.xacro (robot description, xacro)
@@ -4,7 +4,7 @@
                          	Misc
      ========================================================= -->
-	<xacro:include filename="$(find terrasentia_sensors)/urdf/gps/gps.urdf.xacro" />
-	<xacro:include filename="$(find terrasentia_sensors)/urdf/gps/gps_quad.urdf.xacro" />
-	<xacro:include filename="$(find terrasentia_sensors)/urdf/gps/gps_with_mast.urdf.xacro" />
-	<xacro:include filename="$(find terrasentia_sensors)/urdf/gps/gps-with-periodicnoisebox.urdf.xacro" />
+	<xacro:include filename="$(find gazebo_sensor_collection)/urdf/gps/gps_standard.urdf.xacro" />
+	<xacro:include filename="$(find gazebo_sensor_collection)/urdf/gps/gps_quad.urdf.xacro" />
+	<xacro:include filename="$(find gazebo_sensor_collection)/urdf/gps/gps_with_mast.urdf.xacro" />
+	<xacro:include filename="$(find gazebo_sensor_collection)/urdf/gps/gps_with_dropout.urdf.xacro" />
 </robot>

File: urdf/gps/gps_standard.urdf.xacro (robot description, xacro)
@@ -1,7 +1,6 @@
 <?xml version="1.0"?>
-<robot name="sensor_gps_with_dropout" xmlns:xacro="http://ros.org/wiki/xacro">
-	<xacro:include filename="$(find terrasentia_sensors)/urdf/includes/materials.urdf.xacro"/>
-	<xacro:include filename="$(find terrasentia_world)/urdf/includes/macros.urdf.xacro"/>
-  	<xacro:macro name="sensor_gps_with_dropout" params="name parent *origin color ref_lat ref_long ref_head drift vel_drift noise vel_noise update_rate">
+<robot name="sensor_standard_gps" xmlns:xacro="http://ros.org/wiki/xacro">
+	<xacro:include filename="$(find gazebo_sensor_collection)/urdf/includes/materials.urdf.xacro"/>
+  	<xacro:macro name="sensor_standard_gps" params="name parent *origin color ref_lat ref_long ref_head drift vel_drift noise vel_noise update_rate">
 		<joint name="${name}_joint" type="fixed">
 			<axis xyz="0 1 0"/>
@@ -19,5 +18,5 @@
 				<origin rpy="0 0 0" xyz="0 0 0"/>
 				<geometry>
-					<mesh filename="package://terrasentia_sensors/meshes/antenna_3GO16.stl" scale="1.0 1.0 1.0"/>
+					<mesh filename="package://gazebo_sensor_collection/meshes/gps/antenna_3GO16.stl" scale="1.0 1.0 1.0"/>
 				</geometry>
 				<xacro:color_material color="${color}"/>
@@ -26,5 +25,5 @@
 				<origin rpy="0 0 0" xyz="0 0 0"/>
 				<geometry>
-					<mesh filename="package://terrasentia_sensors/meshes/antenna_3GO16.stl" scale="1.0 1.0 1.0"/>
+					<mesh filename="package://gazebo_sensor_collection/meshes/gps/antenna_3GO16.stl" scale="1.0 1.0 1.0"/>
 				</geometry>
 			</collision>
@@ -35,17 +34,14 @@
 		<xacro:color_gazebo parent="${name}_link" color="${color}"/>
 		<gazebo>
-			<plugin name="${name}_controller" filename="libterra_ros_gps_with_dropout.so">
-				<xacro:include filename="$(find terrasentia_sensors)/config/gps/custom_gps_behavior.geofence"/>
-				<xacro:include filename="$(find terrasentia_sensors)/config/gps/plots.xacro"/>
+			<plugin name="${name}_controller" filename="libgazebo_ros_gps.so">
 				<alwaysOn>1</alwaysOn>
 				<updateRate>${update_rate}</updateRate>
-				<bodyName>${name}_link</bodyName> <!-- must be the link of the gps device, not the base_link or base_footprint -->
+				<bodyName>${name}_link</bodyName>
 				<frameId>${name}_link</frameId>
-				<topicName>terra/${name}/fix</topicName>
-				<velocityTopicName>terra/${name}/fix_velocity</velocityTopicName>
-				<terraTopicName>terra/${name}</terraTopicName>
+				<topicName>/${name}</topicName>
 				<referenceLatitude>${ref_lat}</referenceLatitude>
 				<referenceLongitude>${ref_long}</referenceLongitude>
 				<referenceHeading>${ref_head}</referenceHeading>
+				<velocityTopicName>${name}/fix_velocity</velocityTopicName>
 				<drift>${drift} ${drift} ${drift}</drift>
 				<gaussianNoise>${noise} ${noise} ${noise}</gaussianNoise>

File: urdf/gps/gps_with_mast.urdf.xacro (robot description, xacro)
@@ -46,5 +46,5 @@
                     <origin rpy="0 0 0" xyz="0 0 0"/>
                     <geometry>
-                         <mesh filename="package://terrasentia_sensors/meshes/antenna_3GO16.stl" scale="1.0 1.0 1.0"/>
+                         <mesh filename="package://gazebo_sensor_collection/meshes/gps/antenna_3GO16.stl" scale="1.0 1.0 1.0"/>
                     </geometry>
                     <xacro:color_material color="${color}"/>
@@ -53,5 +53,5 @@
                     <origin rpy="0 0 0" xyz="0 0 0"/>
                     <geometry>
-                         <mesh filename="package://terrasentia_sensors/meshes/antenna_3GO16.stl" scale="1.0 1.0 1.0"/>
+                         <mesh filename="package://gazebo_sensor_collection/meshes/gps/antenna_3GO16.stl" scale="1.0 1.0 1.0"/>
                     </geometry>
                </collision>

File: urdf/lidars/hdl_32e.urdf.xacro (robot description, xacro)
@@ -18,5 +18,5 @@
       <visual>
         <geometry>
-          <mesh filename="package://terrasentia_sensors/meshes/HDL32E_base.dae" />
+          <mesh filename="package://gazebo_sensor_collection/meshes/lidars/velodyne/HDL32E_base.dae" />
         </geometry>
       </visual>
@@ -42,5 +42,5 @@
         <origin xyz="0 0 -0.09081" rpy="0 0 0" />
         <geometry>
-          <mesh filename="package://terrasentia_sensors/meshes/HDL32E_scan.dae" />
+          <mesh filename="package://gazebo_sensor_collection/meshes/lidars/velodyne/HDL32E_scan.dae" />
         </geometry>
       </visual>
