Commit message: fixed references in urdf files. renamed urdf files and internals. mesh directory restructured

File: urdf/lidars/hokuyo3d.urdf.xacro (robot description, xacro)
@@ -1,5 +1,5 @@
 <?xml version="1.0"?>
 <robot name="sensor_hokuyo3d" xmlns:xacro="http://ros.org/wiki/xacro">
-     <xacro:include filename="$(find terrasentia_sensors)/urdf/includes/materials.urdf.xacro"/>
+     <xacro:include filename="$(find gazebo_sensor_collection)/urdf/includes/materials.urdf.xacro"/>
      <xacro:macro name="sensor_hokuyo3d" params="name visualize:=false parent *origin color">
           <joint name="${name}_fix_joint" type="fixed">
@@ -18,5 +18,5 @@
                     <origin xyz="0 0 0" rpy="0 0 0"/>
                     <geometry>
-                         <mesh filename="package://terrasentia_sensors/meshes/hokuyo3d.stl"/>
+                         <mesh filename="package://gazebo_sensor_collection/meshes/lidars/hokuyo/hokuyo3d.stl"/>
                     </geometry>
                     <xacro:color_material color="${color}"/>
@@ -73,6 +73,5 @@
                          </noise>
                     </ray>
-                    <!-- <plugin name="${name}_controller" filename="libgazebo_ros_block_laser.so"> -->
-                    <plugin name="${name}_controller" filename="libterra_ros_3d_gpu_laser.so">
+                    <plugin name="${name}_controller" filename="libgazebo_ros_gpu_laser.so">
                          <topicName>${name}/points</topicName>
                          <frameName>${name}_link</frameName>

File: urdf/lidars/hokuyo_urg04lx.urdf.xacro (robot description, xacro)
@@ -1,5 +1,5 @@
 <?xml version="1.0"?>
 <robot name="sensor_hokuyo_urg04lx" xmlns:xacro="http://ros.org/wiki/xacro">
-	<xacro:include filename="$(find terrasentia_sensors)/urdf/includes/materials.urdf.xacro"/>
+	<xacro:include filename="$(find gazebo_sensor_collection)/urdf/includes/materials.urdf.xacro"/>
 	<xacro:macro name="sensor_hokuyo_urg04lx" params="name visualize:=false parent *origin color min_angle:=-2.0943 max_angle:=2.0943">
 		<joint name="${name}_joint" type="fixed">
@@ -18,5 +18,5 @@
 				<origin xyz="0 0 -0.05" rpy="0 0 0"/>
 				<geometry>
-					<mesh filename="package://terrasentia_sensors/meshes/hokuyo_urg_04lx.dae"/>
+					<mesh filename="package://gazebo_sensor_collection/meshes/lidars/hokuyo/hokuyo_urg_04lx.dae"/>
 				</geometry>
 				<xacro:color_material color="${color}"/>

File: urdf/lidars/hokuyo_ust10lx.urdf.xacro (robot description, xacro)
@@ -1,5 +1,5 @@
 <?xml version="1.0"?>
 <robot name="sensor_hokuyo_ust10lx" xmlns:xacro="http://ros.org/wiki/xacro">
-	<xacro:include filename="$(find terrasentia_sensors)/urdf/includes/materials.urdf.xacro"/>
+	<xacro:include filename="$(find gazebo_sensor_collection)/urdf/includes/materials.urdf.xacro"/>
 	<xacro:macro name="sensor_hokuyo_ust10lx" params="name visualize:=false parent *origin color min_angle:=-2.3562 max_angle:=2.3562">
 		<joint name="${name}_joint" type="fixed">
@@ -18,5 +18,5 @@
 				<origin xyz="0 0 -0.05" rpy="0 0 0"/>
 				<geometry>
-					<mesh filename="package://terrasentia_sensors/meshes/hokuyo_ust_10lx.dae"/>
+					<mesh filename="package://gazebo_sensor_collection/meshes/lidars/hokuyo/hokuyo_ust_10lx.dae"/>
 				</geometry>
 				<xacro:color_material color="${color}"/>
@@ -64,5 +64,5 @@
 				</ray>
 				<plugin name="${name}_controller" filename="libgazebo_ros_gpu_laser.so">
-					<topicName>terra/${name}</topicName>
+					<topicName>${name}/scan</topicName>
 					<frameName>${name}_link</frameName>
 				</plugin>
