Commit message: minor filename changes. updated README. additions for launching test environment.

File: urdf/motion/motion_sensors.urdf.xacro (robot description, xacro)
@@ -13,4 +13,4 @@
 	<xacro:include filename="$(find gazebo_sensor_collection)/urdf/motion/imu_quad.urdf.xacro" />
 	<!-- Rotary Encoder -->
-	<xacro:include filename="$(find gazebo_sensor_collection)/urdf/motion/encoder.urdf.xacro" />
+	<xacro:include filename="$(find gazebo_sensor_collection)/urdf/motion/rotary_encoder.urdf.xacro" />
 </robot>

File: urdf/motion/rotary_encoder.urdf.xacro (robot description, xacro)
@@ -1,5 +1,5 @@
 <?xml version="1.0"?>
 <robot xmlns:xacro="http://ros.org/wiki/xacro">
-     <xacro:macro name="sensor_encoder" params="ns:=/ parent joint:=front_left_wheel_rev d:=0.15 topic:=/encoder update_rate:=100.0 ppr:=150">
+     <xacro:macro name="sensor_rotary_encoder" params="ns:=/ parent joint:=front_left_wheel_rev d:=0.15 topic:=/encoder update_rate:=100.0 ppr:=150">
           <link name="${parent}_encoder_link">
 			<collision>
