Commit message: validated successful loading of a subset of sensors (r200, gps w/ dropout, battery, imu mod, and ust10lx)

File: launch/include/sensors_attachments.urdf.xacro (robot description, xacro)
@@ -1,4 +1,4 @@
 <?xml version="1.0" ?>
-<robot xmlns:xacro="http://ros.org/wiki/xacro">
+<robot name="sensor_suite" xmlns:xacro="http://ros.org/wiki/xacro">
      <!-- ====================================================
           Include Sensor Database for Available Sensors

File: urdf/gps/gps_with_dropout.urdf.xacro (robot description, xacro)
@@ -75,7 +75,7 @@
 				<bodyName>${name}_link</bodyName>
 				<frameId>${name}_link</frameId>
-				<topicName>terra/${name}/fix</topicName>
-				<velocityTopicName>terra/${name}/fix_velocity</velocityTopicName>
-				<terraTopicName>terra/${name}</terraTopicName>
+				<topicName>/${name}/fix</topicName>
+				<velocityTopicName>/${name}/fix_velocity</velocityTopicName>
+				<dataTopicName>/${name}</dataTopicName>
 				<referenceLatitude>${ref_lat}</referenceLatitude>
 				<referenceLongitude>${ref_long}</referenceLongitude>

File: urdf/misc/approximate_battery.urdf.xacro (robot description, xacro)
@@ -1,5 +1,5 @@
 <?xml version="1.0"?>
 <robot xmlns:xacro="http://ros.org/wiki/xacro">
-     <xacro:macro name="sensor_battery_approx" params="ns:=/ name:=5200mAh_LiPo parent:=base_footprint link:=main_battery topic:=terra/battery update_rate:=100.0 tau:=1.9499 vMax:=16.0 vMin:=2.0 v0:=14.0 capacity:=5.2 q0:=5.2 m:=-100.1424 b:=12.694">
+     <xacro:macro name="sensor_battery_approx" params="ns:=/ name:=5200mAh_LiPo parent:=base_footprint link:=main_battery topic:=battery update_rate:=100.0 tau:=1.9499 vMax:=16.0 vMin:=2.0 v0:=14.0 capacity:=5.2 q0:=5.2 m:=-100.1424 b:=12.694">
           <gazebo>
                <plugin name="${link}_plugin" filename="libgazebo_ros_battery_simple.so">

File: urdf/motion/imu_hector.urdf.xacro (robot description, xacro)
@@ -36,5 +36,5 @@
                <plugin name="${name}_controller" filename="libhector_gazebo_ros_imu.so">
                     <alwaysOn>true</alwaysOn>
-                    <topicName>terra/${name}</topicName>
+                    <topicName>/${name}</topicName>
                     <serviceName>${name}/service</serviceName>
                     <bodyName>${name}_link</bodyName>

Commit message: updates to d415

File: launch/include/sensors_attachments.urdf.xacro (robot description, xacro)
@@ -16,11 +16,13 @@
      <xacro:world/>
      <!-- LiDAR sensor_hokuyo_ust10lx -->
-     <xacro:sensor_hokuyo_ust10lx name="hokuyo" parent="world_link" color="black" visualize="true">
+     <!-- <xacro:sensor_hokuyo_ust10lx name="hokuyo" parent="world_link" color="black" visualize="true">
           <origin xyz="0.22 0 0.173" rpy="0 0 0"/>
-     </xacro:sensor_hokuyo_ust10lx>
-     <!-- LiDAR sensor_hokuyo_ust10lx -->
-     <xacro:sensor_realsense_r200 parent="world_link">
+     </xacro:sensor_hokuyo_ust10lx> -->
+     <!-- <xacro:sensor_realsense_r200 parent="world_link">
           <origin xyz="0.26 0 0.05" rpy="0 0 0" />
-     </xacro:sensor_realsense_r200>
+     </xacro:sensor_realsense_r200> -->
+     <xacro:sensor_realsense_d415 parent="world_link">
+          <origin xyz="0.26 0 0.05" rpy="0 0 0" />
+     </xacro:sensor_realsense_d415>
      <!-- IMU -->
      <xacro:sensor_modified_imu name="imu" parent="world_link" color="red"

File: urdf/cameras/camera_sensors.urdf.xacro (robot description, xacro)
@@ -27,3 +27,5 @@
 	<!-- Intel Realsense R200 -->
 	<xacro:include filename="$(find gazebo_sensor_collection)/urdf/cameras/rgbd/realsense_r200.urdf.xacro" />
+	<!-- Intel Realsense D415 -->
+	<xacro:include filename="$(find gazebo_sensor_collection)/urdf/cameras/rgbd/realsense_d415.urdf.xacro" />
 </robot>

File: urdf/cameras/rgbd/realsense_d415.urdf.xacro (robot description, xacro)
@@ -1,4 +1,4 @@
 <?xml version="1.0" ?>
-<robot name="sensor_realsense_r200" xmlns:xacro="http://ros.org/wiki/xacro">
+<robot name="sensor_realsense_d415" xmlns:xacro="http://ros.org/wiki/xacro">
      <xacro:macro name="sensor_realsense_d415" params="prefix:='' parent *origin visualize:=false">
           <!-- ============================================================
